Commit message: first real georg style cartesian controller

File: test/2d_base_bot.urdf (robot description, URDF)
Before this commit: robot pointy, 4 links, 3 joints
Joints:
- joint joint_y: type prismatic -> revolute

File: test/fixed.urdf (robot description, URDF)
Before this commit: robot pointy, 4 links, 3 joints
Joints:
- joint joint_y: axis (none) -> 0 1 0; limit (none) -> lower=-1.3 upper=1.4 effort=1.0 velocity=.3; origin xyz=0.0 0.0 1.0 rpy=1.57079632679 1.57079632679 0.0 -> xyz=0.0 0.0 0.0 rpy=0.0 0.0 0.0; type fixed -> prismatic

Commit message: updated tests and fixed bugs

File: test/2d_base_bot.urdf (robot description, URDF)
Before this commit: robot pointy, 4 links, 3 joints
Joints:
- joint joint_x: limit lower=-3 upper=3 effort=1.0 velocity=.2 -> lower=-3 upper=3 effort=1.0 velocity=.5
- joint joint_y: limit lower=-3 upper=3 effort=1.0 velocity=.2 -> lower=-3 upper=3 effort=1.0 velocity=.5; type revolute -> prismatic
- joint rot_z: limit lower=-3 upper=3 effort=1.0 velocity=.2 -> effort=1.0 velocity=.5; type revolute -> continuous
