Commit message: save

File: test/boxy.urdf (robot description, URDF)
Before this commit: robot boxy_description, 84 links, 83 joints
Links:
- removed link neck_look_target_2
- removed link neck_look_target_3
- removed link neck_look_target_4
Joints:
- removed joint head1
- removed joint head2
- removed joint head3
