Commit message: fixed bug in self collision avoidance when base movement is not available

File: test/urdfs/iai_donbot.urdf (robot description, URDF)
Before this commit: robot iai_donbot, 37 links, 36 joints
Links:
- added link charger; collision box size=0.15 0.3 0.38; visual box size=0.15 0.3 0.38
- added link e_stop; collision box size=0.07 0.07 0.1; visual box size=0.07 0.07 0.1
- added link refills_finger
- added link refills_tool_frame
- added link rs_camera_link
- added link switches; collision box size=0.12 0.4 0.45; visual box size=0.12 0.4 0.45
- added link ur5_touchpad; collision box size=0.32 0.06 0.24; visual box size=0.32 0.06 0.24
- added link wlan; collision box size=0.25 0.14 0.05; visual box size=0.25 0.14 0.05
- added link wrist_collision; collision cylinder length=0.08 radius=0.04
- link base_link: geometry collision mesh filename=package://iai_boxy_base_2/meshes/base_lowres.stl; visual mesh filename=package://iai_boxy_base_2/meshes/base.stl
- link camera_holder_link: geometry collision mesh filename=package://iai_donbot_description/meshes/refills_camera_hold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 scale=1 1 1; visual mesh filename=package://iai_donbot_description/meshes/refills_camera_hold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 scale=1 1 1
Joints:
- removed joint ur5_wrist_3_link-tool0_fixed_joint
- added joint charger_joint: type fixed, parent base_link, child charger, origin xyz=0.075 -0.225 0.19 rpy=0 0 0
- added joint e_stop_joint: type fixed, parent base_link, child e_stop, origin xyz=-0.035 -0.0015 0.52 rpy=0 0 0
- added joint refills_finger_joint: type continuous, parent refills_tool_frame, child refills_finger, axis 1 0 0
- added joint refills_tool_frame_joint: type fixed, parent gripper_tool_frame, child refills_tool_frame, origin xyz=0 0 0.037 rpy=0.0 0.0 0.0
- added joint switches_joint: type fixed, parent base_link, child switches, origin xyz=-0.66 -0.225 0.225 rpy=0 0 0
- added joint ur5_touchpad_joint: type fixed, parent base_link, child ur5_touchpad, origin xyz=-0.16 -0.5355 0.38 rpy=0 0 0
- added joint ur5_wrist_3_passive_joint: type fixed, parent ur5_wrist_3_link, child ur5_tool0, origin xyz=0 0 0 rpy=0 0 0
- added joint wlan_joint: type fixed, parent base_link, child wlan, origin xyz=0.05 -0.225 0.405 rpy=0 -0.314 0
- added joint wrist_collision_joint: type fixed, parent adapter_kms40_fwk050_frame_in, child wrist_collision, origin xyz=0 0 -0.005 rpy=0 0 0
- added joint wristcam_to_realsense_joint: type fixed, parent camera_link, child rs_camera_link, origin xyz=-0.017993 -0.107556 0.017699 rpy=6.270618 4.930698 1.578454
- joint arm_base_mounting_joint: origin xyz=-0.165 -0.1815 0.63 rpy=0.0 0.0 0.0 -> xyz=-0.525 -0.424 0.470 rpy=0.0 0.0 0.0; parent base_footprint -> base_link
- joint base_footprint_joint: origin xyz=0.36 0.25 0.16 rpy=0 0 0 -> xyz=0.25525 0.225 0.1616 rpy=0 0 0
- joint gripper_to_camera_joint: origin xyz=0 -0.075 0.035 rpy=0.261799 0 3.14159265359 -> xyz=0.002956 -0.066498 0.060947 rpy=0.204429 6.281375 3.127197
- joint gripper_tool_frame_joint: origin xyz=0 0 0.154 rpy=0 0 0 -> xyz=0 0 0.144 rpy=0 0 0
- joint plate_joint: origin xyz=0.06 0.02 0.62 rpy=0 0 0 -> xyz=-0.300 -0.230 0.460 rpy=0 0 0; parent base_footprint -> base_link
- joint ur5_ee_fixed_joint: origin xyz=0.0 0.0823 0.0 rpy=0.0 0.0 1.57079632679 -> xyz=0.0 0.0 0.0 rpy=0.0 -1.57079632679 1.57079632679
- joint ur5_elbow_joint: axis 0 1 0 -> 0 0 1; origin xyz=0.0 -0.1197 0.425 rpy=0.0 0.0 0.0 -> xyz=-0.425 0 0 rpy=0 0 0
- joint ur5_shoulder_lift_joint: axis 0 1 0 -> 0 0 1; origin xyz=0.0 0.13585 0.0 rpy=0.0 1.57079632679 0.0 -> xyz=0 0 0 rpy=1.570796327 0 0
- joint ur5_shoulder_pan_joint: origin xyz=0.0 0.0 0.089159 rpy=0.0 0.0 0.0 -> xyz=0 0 0.089159 rpy=0 0 3.14159265359
- joint ur5_wrist_1_joint: axis 0 1 0 -> 0 0 1; origin xyz=0.0 0.0 0.39225 rpy=0.0 1.57079632679 0.0 -> xyz=-0.39225 0 0.10915 rpy=0 0 0
- joint ur5_wrist_2_joint: origin xyz=0.0 0.093 0.0 rpy=0.0 0.0 0.0 -> xyz=0 -0.09465 -1.9413039509e-11 rpy=1.570796327 0 0
- joint ur5_wrist_3_joint: axis 0 1 0 -> 0 0 1; origin xyz=0.0 0.0 0.09465 rpy=0.0 0.0 0.0 -> xyz=0 0.0823 -1.68800121668e-11 rpy=1.57079632659 3.14159265359 3.14159265359
