Commit message: new world and world object classes and pybullet implementations of those

File: test/urdfs/2d_base_bot.urdf (robot description, URDF)
Before this commit: robot pointy, 4 links, 3 joints
Links:
- removed link base_link
- added link root_link
Joints:
- joint joint_x: parent base_link -> root_link

Commit message: fixed cmake

File: test/urdfs/2d_base_bot.urdf (robot description, URDF)
Before this commit: robot pointy, 4 links, 3 joints
Links:
- removed link root_link
- added link base_footprint
- link eef: geometry collision box size=0.1 0.1 0.1; visual box size=0.1 0.1 0.1
Joints:
- joint joint_x: parent root_link -> base_footprint

Commit message: giskard will cancel actions servers that take too long to execute

File: test/urdfs/2d_base_bot.urdf (robot description, URDF)
Before this commit: robot pointy, 4 links, 3 joints
Joints:
- joint joint_x: limit lower=-3 upper=3 effort=1.0 velocity=.5 -> lower=-3 upper=3 effort=1.0 velocity=.1
- joint joint_y: limit lower=-3 upper=3 effort=1.0 velocity=.5 -> lower=-3 upper=3 effort=1.0 velocity=.1
- joint rot_z: limit effort=1.0 velocity=.5 -> effort=1.0 velocity=.1
