Commit message: save

File: test/urdfs/pr2.urdf (robot description, URDF)
Before this commit: robot pr2, 97 links, 96 joints
Links:
- removed link l_gripper_l_finger_tip_frame
Joints:
- removed joint l_gripper_joint

Commit message: fixes for melodic urdf parser

File: test/urdfs/pr2.urdf (robot description, URDF)
Before this commit: robot pr2, 97 links, 96 joints
Joints:
- joint base_bellow_joint: origin xyz=-0.29 0 0.8 rpy=0 0 0 -> xyz=-0.29 0.0 0.8 rpy=0.0 0.0 0.0
- joint base_footprint_joint: origin xyz=0 0 0.051 rpy=0 0 0 -> xyz=0.0 0.0 0.051 rpy=0.0 0.0 0.0
- joint base_laser_joint: axis 0 1 0 -> 0.0 1.0 0.0; origin xyz=0.275 0 0.252 rpy=0 0 0 -> xyz=0.275 0.0 0.252 rpy=0.0 0.0 0.0
- joint bl_caster_l_wheel_joint: axis 0 1 0 -> 0.0 1.0 0.0; origin xyz=0 0.049 0 rpy=0 0 0 -> xyz=0.0 0.049 0.0 rpy=0.0 0.0 0.0
- joint bl_caster_r_wheel_joint: axis 0 1 0 -> 0.0 1.0 0.0; origin xyz=0 -0.049 0 rpy=0 0 0 -> xyz=0.0 -0.049 0.0 rpy=0.0 0.0 0.0
- joint bl_caster_rotation_joint: axis 0 0 1 -> 0.0 0.0 1.0; origin xyz=-0.2246 0.2246 0.0282 rpy=0 0 0 -> xyz=-0.2246 0.2246 0.0282 rpy=0.0 0.0 0.0
- joint br_caster_l_wheel_joint: axis 0 1 0 -> 0.0 1.0 0.0; origin xyz=0 0.049 0 rpy=0 0 0 -> xyz=0.0 0.049 0.0 rpy=0.0 0.0 0.0
- joint br_caster_r_wheel_joint: axis 0 1 0 -> 0.0 1.0 0.0; origin xyz=0 -0.049 0 rpy=0 0 0 -> xyz=0.0 -0.049 0.0 rpy=0.0 0.0 0.0
- joint br_caster_rotation_joint: axis 0 0 1 -> 0.0 0.0 1.0; origin xyz=-0.2246 -0.2246 0.0282 rpy=0 0 0 -> xyz=-0.2246 -0.2246 0.0282 rpy=0.0 0.0 0.0
- joint double_stereo_frame_joint: origin xyz=0 0 0 rpy=0 0 0 -> xyz=0.0 0.0 0.0 rpy=0.0 0.0 0.0
- joint fl_caster_l_wheel_joint: axis 0 1 0 -> 0.0 1.0 0.0; origin xyz=0 0.049 0 rpy=0 0 0 -> xyz=0.0 0.049 0.0 rpy=0.0 0.0 0.0
- joint fl_caster_r_wheel_joint: axis 0 1 0 -> 0.0 1.0 0.0; origin xyz=0 -0.049 0 rpy=0 0 0 -> xyz=0.0 -0.049 0.0 rpy=0.0 0.0 0.0
- joint fl_caster_rotation_joint: axis 0 0 1 -> 0.0 0.0 1.0; origin xyz=0.2246 0.2246 0.0282 rpy=0 0 0 -> xyz=0.2246 0.2246 0.0282 rpy=0.0 0.0 0.0
- joint fr_caster_l_wheel_joint: axis 0 1 0 -> 0.0 1.0 0.0; origin xyz=0 0.049 0 rpy=0 0 0 -> xyz=0.0 0.049 0.0 rpy=0.0 0.0 0.0
- joint fr_caster_r_wheel_joint: axis 0 1 0 -> 0.0 1.0 0.0; origin xyz=0 -0.049 0 rpy=0 0 0 -> xyz=0.0 -0.049 0.0 rpy=0.0 0.0 0.0
- joint fr_caster_rotation_joint: axis 0 0 1 -> 0.0 0.0 1.0; origin xyz=0.2246 -0.2246 0.0282 rpy=0 0 0 -> xyz=0.2246 -0.2246 0.0282 rpy=0.0 0.0 0.0
- joint head_mount_joint: origin xyz=-0.138 0 0.091 rpy=0 0 0 -> xyz=-0.138 0.0 0.091 rpy=0.0 0.0 0.0
- joint head_mount_kinect_ir_joint: origin xyz=-0.032267 0.0125 0.136453 rpy=0 0 0 -> xyz=-0.032267 0.0125 0.136453 rpy=0.0 0.0 0.0
- joint head_mount_kinect_ir_optical_frame_joint: origin xyz=0 0.01 0 rpy=-1.57079632679 0 -1.57079632679 -> xyz=0.0 0.01 0.0 rpy=-1.57079632679 0.0 -1.57079632679
- joint head_mount_kinect_rgb_optical_frame_joint: origin xyz=0 0 0 rpy=-1.57079632679 0 -1.57079632679 -> xyz=0.0 0.0 0.0 rpy=-1.57079632679 0.0 -1.57079632679
- joint head_mount_prosilica_joint: origin xyz=-0.046457 0.0125 0.088921 rpy=0 0 0 -> xyz=-0.046457 0.0125 0.088921 rpy=0.0 0.0 0.0
- joint head_mount_prosilica_optical_frame_joint: origin xyz=0 0 0 rpy=-1.57079632679 0 -1.57079632679 -> xyz=0.0 0.0 0.0 rpy=-1.57079632679 0.0 -1.57079632679
- joint head_pan_joint: axis 0 0 1 -> 0.0 0.0 1.0; origin xyz=-0.01707 0 0.38145 rpy=0 0 0 -> xyz=-0.01707 0.0 0.38145 rpy=0.0 0.0 0.0
- joint head_plate_frame_joint: origin xyz=0.0232 0 0.0645 rpy=0 0 0 -> xyz=0.0232 0.0 0.0645 rpy=0.0 0.0 0.0
- joint head_tilt_joint: axis 0 1 0 -> 0.0 1.0 0.0; origin xyz=0.068 0 0 rpy=0 0 0 -> xyz=0.068 0.0 0.0 rpy=0.0 0.0 0.0
- joint high_def_optical_frame_joint: origin xyz=0 0 0 rpy=-1.57079632679 0 -1.57079632679 -> xyz=0.0 0.0 0.0 rpy=-1.57079632679 0.0 -1.57079632679
- joint imu_joint: axis 0 1 0 -> 0.0 1.0 0.0; origin xyz=-0.02977 -0.1497 0.164 rpy=0 3.14159265359 0 -> xyz=-0.02977 -0.1497 0.164 rpy=0.0 3.14159265359 0.0
- joint l_elbow_flex_joint: axis 0 1 0 -> 0.0 1.0 0.0; origin xyz=0.4 0 0 rpy=0 0 0 -> xyz=0.4 0.0 0.0 rpy=0.0 0.0 0.0
- joint l_force_torque_adapter_joint: origin xyz=0.0356 0 0 rpy=0 -1.570796326795 0 -> xyz=0.0356 0.0 0.0 rpy=0.0 -1.570796326795 0.0
- joint l_force_torque_joint: origin xyz=0 0 0 rpy=0 0 1.221730476396 -> xyz=0.0 0.0 0.0 rpy=0.0 0.0 1.221730476396
- joint l_forearm_cam_optical_frame_joint: origin xyz=0 0 0 rpy=-1.57079632679 0 -1.57079632679 -> xyz=0.0 0.0 0.0 rpy=-1.57079632679 0.0 -1.57079632679
- joint l_forearm_joint: origin xyz=0 0 0 rpy=0 0 0 -> xyz=0.0 0.0 0.0 rpy=0.0 0.0 0.0
- joint l_forearm_roll_joint: axis 1 0 0 -> 1.0 0.0 0.0; origin xyz=0 0 0 rpy=0 0 0 -> xyz=0.0 0.0 0.0 rpy=0.0 0.0 0.0
- joint l_gripper_joint: axis 0 1 0 -> 0.0 1.0 0.0; origin xyz=0 0 0 rpy=0 0 0 -> xyz=0.0 0.0 0.0 rpy=0.0 0.0 0.0
- joint l_gripper_l_finger_joint: axis 0 0 1 -> 0.0 0.0 1.0; origin xyz=0.07691 0.01 0 rpy=0 0 0 -> xyz=0.07691 0.01 0.0 rpy=0.0 0.0 0.0
- joint l_gripper_l_finger_tip_joint: axis 0 0 -1 -> 0.0 0.0 -1; origin xyz=0.09137 0.00495 0 rpy=0 0 0 -> xyz=0.09137 0.00495 0.0 rpy=0.0 0.0 0.0
- joint l_gripper_led_joint: origin xyz=0.0513 0 0.0244 rpy=0 0 0 -> xyz=0.0513 0.0 0.0244 rpy=0.0 0.0 0.0
- joint l_gripper_motor_accelerometer_joint: origin xyz=0 0 0 rpy=0 0 0 -> xyz=0.0 0.0 0.0 rpy=0.0 0.0 0.0
- joint l_gripper_motor_screw_joint: axis 0 1 0 -> 0.0 1.0 0.0; origin xyz=0 0 0 rpy=0 0 0 -> xyz=0.0 0.0 0.0 rpy=0.0 0.0 0.0
- joint l_gripper_motor_slider_joint: axis 1 0 0 -> 1.0 0.0 0.0; origin xyz=0.16828 0 0 rpy=0 0 0 -> xyz=0.16828 0.0 0.0 rpy=0.0 0.0 0.0
- joint l_gripper_palm_joint: origin xyz=0 0 0 rpy=0 1.570796326795 -1.221730476396 -> xyz=0.0 0.0 0.0 rpy=0.0 1.570796326795 -1.221730476396
- joint l_gripper_r_finger_joint: axis 0 0 -1 -> 0.0 0.0 -1; origin xyz=0.07691 -0.01 0 rpy=0 0 0 -> xyz=0.07691 -0.01 0.0 rpy=0.0 0.0 0.0
- joint l_gripper_r_finger_tip_joint: axis 0 0 1 -> 0.0 0.0 1.0; origin xyz=0.09137 -0.00495 0 rpy=0 0 0 -> xyz=0.09137 -0.00495 0.0 rpy=0.0 0.0 0.0
- joint l_gripper_tool_joint: origin xyz=0.18 0 0 rpy=0 0 0 -> xyz=0.18 0.0 0.0 rpy=0.0 0.0 0.0
- joint l_shoulder_lift_joint: axis 0 1 0 -> 0.0 1.0 0.0; origin xyz=0.1 0 0 rpy=0 0 0 -> xyz=0.1 0.0 0.0 rpy=0.0 0.0 0.0
- joint l_shoulder_pan_joint: axis 0 0 1 -> 0.0 0.0 1.0; origin xyz=0 0.188 0 rpy=0 0 0 -> xyz=0.0 0.188 0.0 rpy=0.0 0.0 0.0
- joint l_torso_lift_side_plate_joint: origin xyz=0.0535 0.209285 0.176625 rpy=0 0 0 -> xyz=0.0535 0.209285 0.176625 rpy=0.0 0.0 0.0
- joint l_upper_arm_joint: origin xyz=0 0 0 rpy=0 0 0 -> xyz=0.0 0.0 0.0 rpy=0.0 0.0 0.0
- joint l_upper_arm_roll_joint: axis 1 0 0 -> 1.0 0.0 0.0; origin xyz=0 0 0 rpy=0 0 0 -> xyz=0.0 0.0 0.0 rpy=0.0 0.0 0.0
- joint l_wrist_flex_joint: axis 0 1 0 -> 0.0 1.0 0.0; origin xyz=0.321 0 0 rpy=0 0 0 -> xyz=0.321 0.0 0.0 rpy=0.0 0.0 0.0
- joint l_wrist_roll_joint: axis 1 0 0 -> 1.0 0.0 0.0; origin xyz=0 0 0 rpy=0 0 0 -> xyz=0.0 0.0 0.0 rpy=0.0 0.0 0.0
- joint laser_tilt_joint: axis 0 1 0 -> 0.0 1.0 0.0; origin xyz=0 0 0.028389479248 rpy=0 0 -0.007935244203 -> xyz=0.0 0.0 0.028389479248 rpy=0.0 0.0 -0.007935244203
- joint laser_tilt_mount_joint: axis 0 1 0 -> 0.0 1.0 0.0; origin xyz=0.09893 0 0.227 rpy=0 0 0 -> xyz=0.09893 0.0 0.227 rpy=0.0 0.0 0.0
- joint narrow_stereo_l_stereo_camera_frame_joint: origin xyz=0 0 0 rpy=0 0 0 -> xyz=0.0 0.0 0.0 rpy=0.0 0.0 0.0
- joint narrow_stereo_l_stereo_camera_optical_frame_joint: origin xyz=0 0 0 rpy=-1.57079632679 0 -1.57079632679 -> xyz=0.0 0.0 0.0 rpy=-1.57079632679 0.0 -1.57079632679
- joint narrow_stereo_optical_frame_joint: origin xyz=0 0 0 rpy=-1.57079632679 0 -1.57079632679 -> xyz=0.0 0.0 0.0 rpy=-1.57079632679 0.0 -1.57079632679
- joint narrow_stereo_r_stereo_camera_frame_joint: origin xyz=0 -0.09 0 rpy=0 0 0 -> xyz=0.0 -0.09 0.0 rpy=0.0 0.0 0.0
- joint narrow_stereo_r_stereo_camera_optical_frame_joint: origin xyz=0 0 0 rpy=-1.57079632679 0 -1.57079632679 -> xyz=0.0 0.0 0.0 rpy=-1.57079632679 0.0 -1.57079632679
- joint projector_wg6802418_child_frame_joint: origin xyz=0 0 0 rpy=0 -1.57079632679 0 -> xyz=0.0 0.0 0.0 rpy=0.0 -1.57079632679 0.0
- joint projector_wg6802418_frame_joint: origin xyz=0 0.11 0.0546 rpy=0 0 0 -> xyz=0.0 0.11 0.0546 rpy=0.0 0.0 0.0
- joint r_elbow_flex_joint: axis 0 1 0 -> 0.0 1.0 0.0; origin xyz=0.4 0 0 rpy=0 0 0 -> xyz=0.4 0.0 0.0 rpy=0.0 0.0 0.0
- joint r_forearm_cam_optical_frame_joint: origin xyz=0 0 0 rpy=-1.57079632679 0 -1.57079632679 -> xyz=0.0 0.0 0.0 rpy=-1.57079632679 0.0 -1.57079632679
- joint r_forearm_joint: origin xyz=0 0 0 rpy=0 0 0 -> xyz=0.0 0.0 0.0 rpy=0.0 0.0 0.0
- joint r_forearm_roll_joint: axis 1 0 0 -> 1.0 0.0 0.0; origin xyz=0 0 0 rpy=0 0 0 -> xyz=0.0 0.0 0.0 rpy=0.0 0.0 0.0
- joint r_gripper_joint: axis 0 1 0 -> 0.0 1.0 0.0; origin xyz=0 0 0 rpy=0 0 0 -> xyz=0.0 0.0 0.0 rpy=0.0 0.0 0.0
- joint r_gripper_l_finger_joint: axis 0 0 1 -> 0.0 0.0 1.0; origin xyz=0.07691 0.01 0 rpy=0 0 0 -> xyz=0.07691 0.01 0.0 rpy=0.0 0.0 0.0
- joint r_gripper_l_finger_tip_joint: axis 0 0 -1 -> 0.0 0.0 -1; origin xyz=0.09137 0.00495 0 rpy=0 0 0 -> xyz=0.09137 0.00495 0.0 rpy=0.0 0.0 0.0
- joint r_gripper_led_joint: origin xyz=0.0513 0 0.0244 rpy=0 0 0 -> xyz=0.0513 0.0 0.0244 rpy=0.0 0.0 0.0
- joint r_gripper_motor_accelerometer_joint: origin xyz=0 0 0 rpy=0 0 0 -> xyz=0.0 0.0 0.0 rpy=0.0 0.0 0.0
- joint r_gripper_motor_screw_joint: axis 0 1 0 -> 0.0 1.0 0.0; origin xyz=0 0 0 rpy=0 0 0 -> xyz=0.0 0.0 0.0 rpy=0.0 0.0 0.0
- joint r_gripper_motor_slider_joint: axis 1 0 0 -> 1.0 0.0 0.0; origin xyz=0.16828 0 0 rpy=0 0 0 -> xyz=0.16828 0.0 0.0 rpy=0.0 0.0 0.0
- joint r_gripper_palm_joint: origin xyz=0 0 0 rpy=0 0 0 -> xyz=0.0 0.0 0.0 rpy=0.0 0.0 0.0
- joint r_gripper_r_finger_joint: axis 0 0 -1 -> 0.0 0.0 -1; origin xyz=0.07691 -0.01 0 rpy=0 0 0 -> xyz=0.07691 -0.01 0.0 rpy=0.0 0.0 0.0
- joint r_gripper_r_finger_tip_joint: axis 0 0 1 -> 0.0 0.0 1.0; origin xyz=0.09137 -0.00495 0 rpy=0 0 0 -> xyz=0.09137 -0.00495 0.0 rpy=0.0 0.0 0.0
- joint r_gripper_tool_joint: origin xyz=0.18 0 0 rpy=0 0 0 -> xyz=0.18 0.0 0.0 rpy=0.0 0.0 0.0
- joint r_shoulder_lift_joint: axis 0 1 0 -> 0.0 1.0 0.0; origin xyz=0.1 0 0 rpy=0 0 0 -> xyz=0.1 0.0 0.0 rpy=0.0 0.0 0.0
- joint r_shoulder_pan_joint: axis 0 0 1 -> 0.0 0.0 1.0; origin xyz=0 -0.188 0 rpy=0 0 0 -> xyz=0.0 -0.188 0.0 rpy=0.0 0.0 0.0
- joint r_torso_lift_side_plate_joint: origin xyz=0.0535 -0.209285 0.176625 rpy=0 0 0 -> xyz=0.0535 -0.209285 0.176625 rpy=0.0 0.0 0.0
- joint r_upper_arm_joint: origin xyz=0 0 0 rpy=0 0 0 -> xyz=0.0 0.0 0.0 rpy=0.0 0.0 0.0
- joint r_upper_arm_roll_joint: axis 1 0 0 -> 1.0 0.0 0.0; origin xyz=0 0 0 rpy=0 0 0 -> xyz=0.0 0.0 0.0 rpy=0.0 0.0 0.0
- joint r_wrist_flex_joint: axis 0 1 0 -> 0.0 1.0 0.0; origin xyz=0.321 0 0 rpy=0 0 0 -> xyz=0.321 0.0 0.0 rpy=0.0 0.0 0.0
- joint r_wrist_roll_joint: axis 1 0 0 -> 1.0 0.0 0.0; origin xyz=0 0 0 rpy=0 0 0 -> xyz=0.0 0.0 0.0 rpy=0.0 0.0 0.0
- joint sensor_mount_frame_joint: origin xyz=0 0 0 rpy=0 0 0 -> xyz=0.0 0.0 0.0 rpy=0.0 0.0 0.0
- joint torso_lift_joint: axis 0 0 1 -> 0.0 0.0 1.0; origin xyz=-0.05 0 0.739675 rpy=0 0 0 -> xyz=-0.05 0.0 0.739675 rpy=0.0 0.0 0.0
- joint torso_lift_motor_screw_joint: axis 0 0 1 -> 0.0 0.0 1.0; origin xyz=-0.15 0 0.7 rpy=0 0 0 -> xyz=-0.15 0.0 0.7 rpy=0.0 0.0 0.0
- joint wide_stereo_l_stereo_camera_frame_joint: origin xyz=0 0 0 rpy=0 0 0 -> xyz=0.0 0.0 0.0 rpy=0.0 0.0 0.0
- joint wide_stereo_l_stereo_camera_optical_frame_joint: origin xyz=0 0 0 rpy=-1.57079632679 0 -1.57079632679 -> xyz=0.0 0.0 0.0 rpy=-1.57079632679 0.0 -1.57079632679
- joint wide_stereo_optical_frame_joint: origin xyz=0 0 0 rpy=-1.57079632679 0 -1.57079632679 -> xyz=0.0 0.0 0.0 rpy=-1.57079632679 0.0 -1.57079632679
- joint wide_stereo_r_stereo_camera_frame_joint: origin xyz=0 -0.09 0 rpy=0 0 0 -> xyz=0.0 -0.09 0.0 rpy=0.0 0.0 0.0
- joint wide_stereo_r_stereo_camera_optical_frame_joint: origin xyz=0 0 0 rpy=-1.57079632679 0 -1.57079632679 -> xyz=0.0 0.0 0.0 rpy=-1.57079632679 0.0 -1.57079632679

Commit message: implemented proxsuite

File: test/urdfs/pr2.urdf (robot description, URDF)
Before this commit: robot pr2, 97 links, 96 joints
Links:
- link base_link: geometry collision mesh filename=package://iai_pr2_description/meshes/base_v0/base_L.stl; visual mesh filename=package://iai_pr2_description/meshes/base_v0/base.dae
- link bl_caster_l_wheel_link: geometry collision cylinder length=0.034 radius=0.074792; visual mesh filename=package://iai_pr2_description/meshes/base_v0/wheel.dae
- link bl_caster_r_wheel_link: geometry collision cylinder length=0.034 radius=0.074792; visual mesh filename=package://iai_pr2_description/meshes/base_v0/wheel.dae
- link bl_caster_rotation_link: geometry collision mesh filename=package://iai_pr2_description/meshes/base_v0/caster_L.stl; visual mesh filename=package://iai_pr2_description/meshes/base_v0/caster.stl
- link br_caster_l_wheel_link: geometry collision cylinder length=0.034 radius=0.074792; visual mesh filename=package://iai_pr2_description/meshes/base_v0/wheel.dae
- link br_caster_r_wheel_link: geometry collision cylinder length=0.034 radius=0.074792; visual mesh filename=package://iai_pr2_description/meshes/base_v0/wheel.dae
- link br_caster_rotation_link: geometry collision mesh filename=package://iai_pr2_description/meshes/base_v0/caster_L.stl; visual mesh filename=package://iai_pr2_description/meshes/base_v0/caster.stl
- link fl_caster_l_wheel_link: geometry collision cylinder length=0.034 radius=0.074792; visual mesh filename=package://iai_pr2_description/meshes/base_v0/wheel.dae
- link fl_caster_r_wheel_link: geometry collision cylinder length=0.034 radius=0.074792; visual mesh filename=package://iai_pr2_description/meshes/base_v0/wheel.dae
- link fl_caster_rotation_link: geometry collision mesh filename=package://iai_pr2_description/meshes/base_v0/caster_L.stl; visual mesh filename=package://iai_pr2_description/meshes/base_v0/caster.stl
- link fr_caster_l_wheel_link: geometry collision cylinder length=0.034 radius=0.074792; visual mesh filename=package://iai_pr2_description/meshes/base_v0/wheel.dae
- link fr_caster_r_wheel_link: geometry collision cylinder length=0.034 radius=0.074792; visual mesh filename=package://iai_pr2_description/meshes/base_v0/wheel.dae
- link fr_caster_rotation_link: geometry collision mesh filename=package://iai_pr2_description/meshes/base_v0/caster_L.stl; visual mesh filename=package://iai_pr2_description/meshes/base_v0/caster.stl
- link head_mount_link: geometry collision sphere radius=0.0005; visual mesh filename=package://iai_pr2_description/meshes/sensors/kinect_prosili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 scale=0.001 0.001 0.001
- link head_pan_link: geometry collision mesh filename=package://iai_pr2_description/meshes/head_v0/head_pan_L.stl; visual mesh filename=package://iai_pr2_description/meshes/head_v0/head_pan.dae
- link head_tilt_link: geometry collision mesh filename=package://iai_pr2_description/meshes/head_v0/head_tilt_L.stl; visual mesh filename=package://iai_pr2_description/meshes/head_v0/head_tilt.dae
- link l_elbow_flex_link: geometry collision mesh filename=package://iai_pr2_description/meshes/upper_arm_v0/elbow_fle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; visual mesh filename=package://iai_pr2_description/meshes/upper_arm_v0/elbow_fle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
- link l_forearm_link: geometry collision mesh filename=package://iai_pr2_description/meshes/forearm_v0/forearm.stl; visual mesh filename=package://iai_pr2_description/meshes/forearm_v0/forearm.dae
- link l_forearm_roll_link: geometry collision mesh filename=package://iai_pr2_description/meshes/upper_arm_v0/forearm_r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; visual mesh filename=package://iai_pr2_description/meshes/upper_arm_v0/forearm_r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
- link l_gripper_l_finger_link: geometry collision mesh filename=package://iai_pr2_description/meshes/gripper_v0/l_finger.stl; visual mesh filename=package://iai_pr2_description/meshes/gripper_v0/l_finger.dae
- link l_gripper_l_finger_tip_link: geometry collision mesh filename=package://iai_pr2_description/meshes/gripper_v0/l_finger_ti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; visual mesh filename=package://iai_pr2_description/meshes/gripper_v0/l_finger_ti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
- link l_gripper_palm_link: geometry collision mesh filename=package://iai_pr2_description/meshes/gripper_v0/gripper_pal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; visual mesh filename=package://iai_pr2_description/meshes/gripper_v0/gripper_pal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
- link l_gripper_r_finger_link: geometry collision mesh filename=package://iai_pr2_description/meshes/gripper_v0/l_finger.stl; visual mesh filename=package://iai_pr2_description/meshes/gripper_v0/l_finger.dae
- link l_gripper_r_finger_tip_link: geometry collision mesh filename=package://iai_pr2_description/meshes/gripper_v0/l_finger_ti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; visual mesh filename=package://iai_pr2_description/meshes/gripper_v0/l_finger_ti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
- link l_shoulder_lift_link: geometry collision mesh filename=package://iai_pr2_description/meshes/shoulder_v0/shoulder_l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; visual mesh filename=package://iai_pr2_description/meshes/shoulder_v0/shoulder_l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
- link l_shoulder_pan_link: geometry collision mesh filename=package://iai_pr2_description/meshes/shoulder_v0/shoulder_p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; visual mesh filename=package://iai_pr2_description/meshes/shoulder_v0/shoulder_p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
- link l_upper_arm_link: geometry collision mesh filename=package://iai_pr2_description/meshes/upper_arm_v0/upper_arm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; visual mesh filename=package://iai_pr2_description/meshes/upper_arm_v0/upper_arm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
- link l_upper_arm_roll_link: geometry collision mesh filename=package://iai_pr2_description/meshes/shoulder_v0/upper_arm_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; visual mesh filename=package://iai_pr2_description/meshes/shoulder_v0/upper_arm_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
- link l_wrist_flex_link: geometry collision mesh filename=package://iai_pr2_description/meshes/forearm_v0/wrist_flex.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; visual mesh filename=package://iai_pr2_description/meshes/forearm_v0/wrist_flex.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
- link l_wrist_roll_link: geometry collision mesh filename=package://iai_pr2_description/meshes/forearm_v0/wrist_roll_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; visual mesh filename=package://iai_pr2_description/meshes/forearm_v0/wrist_roll.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
- link laser_tilt_mount_link: geometry collision mesh filename=package://iai_pr2_description/meshes/tilting_laser_v0/tilti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; visual mesh filename=package://iai_pr2_description/meshes/tilting_laser_v0/tilti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
- link r_elbow_flex_link: geometry collision mesh filename=package://iai_pr2_description/meshes/upper_arm_v0/elbow_fle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; visual mesh filename=package://iai_pr2_description/meshes/upper_arm_v0/elbow_fle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
- link r_forearm_link: geometry collision mesh filename=package://iai_pr2_description/meshes/forearm_v0/forearm.stl; visual mesh filename=package://iai_pr2_description/meshes/forearm_v0/forearm.dae
- link r_forearm_roll_link: geometry collision mesh filename=package://iai_pr2_description/meshes/upper_arm_v0/forearm_r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; visual mesh filename=package://iai_pr2_description/meshes/upper_arm_v0/forearm_r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
- link r_gripper_l_finger_link: geometry collision mesh filename=package://iai_pr2_description/meshes/gripper_v0/l_finger.stl; visual mesh filename=package://iai_pr2_description/meshes/gripper_v0/l_finger.dae
- link r_gripper_l_finger_tip_link: geometry collision mesh filename=package://iai_pr2_description/meshes/gripper_v0/l_finger_ti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; visual mesh filename=package://iai_pr2_description/meshes/gripper_v0/l_finger_ti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
- link r_gripper_palm_link: geometry collision mesh filename=package://iai_pr2_description/meshes/gripper_v0/gripper_pal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; visual mesh filename=package://iai_pr2_description/meshes/gripper_v0/gripper_pal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
- link r_gripper_r_finger_link: geometry collision mesh filename=package://iai_pr2_description/meshes/gripper_v0/l_finger.stl; visual mesh filename=package://iai_pr2_description/meshes/gripper_v0/l_finger.dae
- link r_gripper_r_finger_tip_link: geometry collision mesh filename=package://iai_pr2_description/meshes/gripper_v0/l_finger_ti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; visual mesh filename=package://iai_pr2_description/meshes/gripper_v0/l_finger_ti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
- link r_shoulder_lift_link: geometry collision mesh filename=package://iai_pr2_description/meshes/shoulder_v0/shoulder_l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; visual mesh filename=package://iai_pr2_description/meshes/shoulder_v0/shoulder_l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
- link r_shoulder_pan_link: geometry collision mesh filename=package://iai_pr2_description/meshes/shoulder_v0/shoulder_p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; visual mesh filename=package://iai_pr2_description/meshes/shoulder_v0/shoulder_p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
- link r_upper_arm_link: geometry collision mesh filename=package://iai_pr2_description/meshes/upper_arm_v0/upper_arm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; visual mesh filename=package://iai_pr2_description/meshes/upper_arm_v0/upper_arm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
- link r_upper_arm_roll_link: geometry collision mesh filename=package://iai_pr2_description/meshes/shoulder_v0/upper_arm_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; visual mesh filename=package://iai_pr2_description/meshes/shoulder_v0/upper_arm_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
- link r_wrist_flex_link: geometry collision mesh filename=package://iai_pr2_description/meshes/forearm_v0/wrist_flex.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; visual mesh filename=package://iai_pr2_description/meshes/forearm_v0/wrist_flex.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
- link r_wrist_roll_link: geometry collision mesh filename=package://iai_pr2_description/meshes/forearm_v0/wrist_roll_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; visual mesh filename=package://iai_pr2_description/meshes/forearm_v0/wrist_roll.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
- link torso_lift_link: geometry collision mesh filename=package://iai_pr2_description/meshes/torso_v0/torso_lift_L.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; visual mesh filename=package://iai_pr2_description/meshes/torso_v0/torso_lift.dae
