Commit message: fixed feature functions python interface call and spoon test

File: test/spoon/urdf/spoon.urdf (robot description, URDF)
Before this commit: robot spoon, 1 links, 0 joints
Links:
- link spoon: geometry collision mesh filename=package://giskardpy_ros/test/spoon/meshes/stl/SM_Spoon_1.stl; collision mesh filename=package://giskardpy_ros/test/spoon/meshes/stl/SM_Spoon_10.s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
